File: Ardu2/design/POC-3_MAX395/KicadProjects/fullCircuit.sch (KiCad schematic (older format))
At the start: 130 parts

Commit message: initial Kicad schematic of full circuit
Parts:
- removed C? (x3): C, symbol C
- removed R? (x5): R, symbol R
- added L?: INDUCTOR, symbol INDUCTOR
- added P? (x5): CONN_01X03, symbol CONN_01X03
- added P?: CONN_01X02, symbol CONN_01X02
- added U?: Pyboard, MODULE, symbol Pyboard
- C? (x2): value CP -> 470µF
- C? (x2): value CP -> 220µF
- D?: value D_Schottky -> 1N5825
- D?: value D_Schottky -> 1N5285
- R? (x2): value R -> 1K
- R? (x2): value R -> 330
Connections:
- net BATin: now reaches U?.1 (+Vin)
- net BATin: now also C?.1, C?.1, U?.1 (+Vin)
- net at U?.2 (Out): now also D?.1 (K), L?.1 (x2)
- net GND: now reaches U?.3 (GND)
- net GND: now also C?.1, C?.2, C?.2, D?.2 (A), L?.2, R?.1, R?.2, U?.5 (~On~/Off)
- net at U?.4 (FB): now also R?.1, R?.2 (x2)
- net V-: now reaches U?.3 (GND)
- net V-: now also C?.2, C?.2, D?.2 (A), R?.2, U?.5 (~On~/Off)
- net V+: now reaches C?.1
- net V+: now also L?.2, R?.1
Other:
- moved on the sheet: C?, D?, L?, R?, U?

Commit message: first full KICAD schematic
Parts:
- removed C? (x23): C, symbol C
- removed R? (x49): R, symbol R
- removed U? (x6): MAX395, MODULE, symbol MAX395
- added C10, C16, C24, C32, C41: 10nF, symbol C
- added C17, C18, C20, C21, C25, C26, C29, C30, C33, C34, C37, C38: 100nF, symbol C
- added C23, C31, C39, C46, C5: 180pF, symbol C
- added R10, R20, R21, R22, R23, R24, R29, R30, R31, R32, R33, R38, R39, R40, R41, R42, R47, R48, R49, R50, R51, R6, R7, R8, R9: 100K, symbol R
- added R11, R19, R28, R37, R46: 64K, symbol R
- added R12, R18, R27, R36, R45: 32K, symbol R
- added R13, R14, R16, R17, R25, R26, R34, R35, R43, R44: 16K, symbol R
- added R15: 22K, symbol R
- added U11, U12, U14, U15, U8, U9: MAX395, MODULE, symbol MAX395
- C11: renamed from C?; value C -> 6.3nF
- C12: renamed from C?; value C -> 4nF
- C13: renamed from C?; value C -> 2nF
- C14: renamed from C?; value C -> 1nF
- C15, C19, C22, C28, C35, C36, C40, C42, C43, C44, C45, C6, C7, C8, C9: renamed from C?; value C -> 100nF
- L3: renamed from L?; value INDUCTOR -> 1mH
- R1: renamed from R?; value R -> 200
- gave numbers to parts that had none: 31
Connections:
- net labels added: A+, A-, AOut+, AOut-, B+, B-, BOut+, BOut-, Batin, C+, C-, COut+, COut-, D+, D-, DOut+, DOut-, MIn+, MIn-, OUT+, OUT-
- wire segments 33 -> 762
- no-connect marks 0 -> 1
Other:
- moved on the sheet: C11, C12, C13, C14, C42, C43, C44, C45, C6, C7, C8, C9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

Commit message: first draft kicad circuit
Parts:
- C1, C2, C3, C4: footprint (none) -> Capacitors_ThroughHole:C_Radial_D10_L16_P5
- C10, C14, C16, C24, C32, C41: footprint (none) -> Capacitors_ThroughHole:C_Disc_D6_P5
- C11: value 6.3nF -> 6.8nF; footprint (none) -> Capacitors_ThroughHole:C_Disc_D6_P5
- C12: value 4nF -> 4.7nF; footprint (none) -> Capacitors_ThroughHole:C_Disc_D6_P5
- C13: value 2nF -> 2.2nF; footprint (none) -> Capacitors_ThroughHole:C_Disc_D6_P5
- C15, C17, C18, C19, C20, C21, C22, C23, C25, C26, C28, C29, C30, C31, C33, C34, C35, C36, C37, C38, C39, C40, C42, C43, C44, C45, C46, C5, C6, C7, C8, C9: footprint (none) -> Capacitors_ThroughHole:C_Disc_D3_P2.5
- C27: value C -> 100nF; footprint (none) -> Capacitors_ThroughHole:C_Disc_D3_P2.5
- D1: value 1N5825 -> 1N5401; footprint (none) -> Diodes_ThroughHole:Diode_DO-201AD_Horizontal_RM15
- D2: value 1N5285 -> 1N5401; footprint (none) -> Diodes_ThroughHole:Diode_DO-201AD_Horizontal_RM15
- L1, L2: footprint (none) -> 330L:330L-Q9N_Inductor
- L3: footprint (none) -> 330L:Inductor
- P1: footprint (none) -> Connect:PINHEAD1-2
- P2, P3, P4, P5, P6: footprint (none) -> Connect:PINHEAD1-3
- R1: value 200 -> 220; footprint (none) -> Resistors_ThroughHole:Resistor_Horizontal_RM10mm
- R10, R13, R14, R15, R16, R17, R2, R20, R21, R22, R23, R24, R25, R26, R29, R3, R30, R31, R32, R33, R34, R35, R38, R39, R4, R40, R41, R42, R43, R44, R47, R48, R49, R5, R50, R51, R6, R7, R8, R9: footprint (none) -> Resistors_ThroughHole:Resistor_Horizontal_RM10mm
- R11, R19, R28, R37, R46: value 64K -> 62K; footprint (none) -> Resistors_ThroughHole:Resistor_Horizontal_RM10mm
- R12, R18, R27, R36, R45: value 32K -> 33K; footprint (none) -> Resistors_ThroughHole:Resistor_Horizontal_RM10mm
- U1: footprint MODULE -> Socket_Strips:Socket_Strip_Straight_1x16
- U10, U11, U12, U13, U14, U15, U16, U17, U18, U5, U6, U7, U8, U9: footprint MODULE -> Housings_DIP:DIP-24__300
- U2, U3: footprint (none) -> NationalSemiconductor:TO263-5
- U4: footprint (none) -> Divers:OPTORESISTOR_NSL-32
Connections:
- wire segments 762 -> 763

Commit message: progress on kicad design
Parts:
- added P?: CONN_01X15, symbol CONN_01X15
- U1: footprint Socket_Strips:Socket_Strip_Straight_1x16 -> 330L:Pyboard16x2
- U2, U3: footprint NationalSemiconductor:TO263-5 -> NationalSemiconductor:T05D
Connections:
- wire segments 763 -> 921
- no-connect marks 1 -> 27

Commit message: working 2 layer kicad pcb
Parts:
- removed P2, P3, P4, P5, P6: CONN_01X03, Connect:PINHEAD1-3, symbol CONN_01X03
- added HS1: HEATSINK, 330L:Heatsink_TO_220_38_20, symbol HEATSINK
- P7: renamed from P?; footprint (none) -> w_conn_pc:DB_15F-VGA
Connections:
- wire segments 921 -> 758
Other:
- moved on the sheet: L3, P7

Commit message: ùore pcb kicad work, mostly failures
Parts:
- removed U4: PHOTORESISTOR, Divers:OPTORESISTOR_NSL-32, symbol PHOTORESISTOR
- added U4: Vactrol, 330L:Vactrol, symbol Vactrol
Connections:
- net labels added: CLK, CS, ShuntControl
- wire segments 758 -> 682
Other:
- moved on the sheet: C1, C10, C11, C12, C13, C14, C15, C16, C17, C18, C19, C2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

Commit message: more pcb experiments
Changed lines of the file:
@@
 Text Label 5150 1000 3    60   ~ 0
 OUT-
+Text Label 6450 1000 3    60   ~ 0
+A+
+Text Label 6350 1000 3    60   ~ 0
+A-
 Text Label 6250 1000 3    60   ~ 0
-A+
+B+
 Text Label 6150 1000 3    60   ~ 0
-A-
-Text Label 6350 1000 3    60   ~ 0
-B+
-Text Label 6450 1000 3    60   ~ 0
 B-
 Text Label 6550 1000 3    60   ~ 0

Commit message: another pcb version...
Changed lines of the file:
@@
 Text Label 2250 3600 0    60   ~ 0
 V+
-NoConn ~ 750  3600
 NoConn ~ 750  3700
 NoConn ~ 750  3800
@@
 	16400 4700 16950 4700
 Wire Wire Line
-	16950 4700 16950 5000
+	16950 5000 16950 4700
 Wire Wire Line
 	16950 4900 16400 4900
 Wire Wire Line
-	16950 5000 16300 5000
+	16300 5000 16950 5000
 Connection ~ 16950 4900
 Wire Wire Line
@@
 	13100 4700 13650 4700
 Wire Wire Line
-	13650 4700 13650 5000
+	13650 5000 13650 4700
 Wire Wire Line
 	13650 4900 13100 4900
 Wire Wire Line
-	13650 5000 13000 5000
+	13000 5000 13650 5000
 Connection ~ 13650 4900
 Wire Wire Line
@@
 	9750 4700 10300 4700
 Wire Wire Line
-	10300 4700 10300 5000
+	10300 5000 10300 4700
 Wire Wire Line
 	10300 4900 9750 4900
 Wire Wire Line
-	10300 5000 9650 5000
+	9650 5000 10300 5000
 Connection ~ 10300 4900
 Wire Wire Line
@@
 	6450 4700 7000 4700
 Wire Wire Line
-	7000 4700 7000 5000
+	7000 5000 7000 4700
 Wire Wire Line
 	7000 4900 6450 4900
 Wire Wire Line
-	7000 5000 6350 5000
+	6350 5000 7000 5000
 Connection ~ 7000 4900
 Wire Wire Line
@@
 	13150 6700 13150 5850
 Wire Wire Line
-	13150 5850 16300 5850
+	16300 5850 13150 5850
 Connection ~ 16300 5850
 Wire Wire Line
@@
 	15650 7100 15600 7100
 Wire Wire Line
-	16300 5850 16300 5000
+	16300 5000 16300 5850
 Connection ~ 15650 6800
 Connection ~ 16350 5900
@@
 Wire Wire Line
 	5650 1400 5650 1000
-Text Label 2250 5100 0    60   ~ 0
+Text Label 750  3600 0    60   ~ 0
 ShuntControl
 Text Label 2250 4600 0    60   ~ 0
@@
 Wire Wire Line
 	1850 850  1550 850
+Text Label 5750 1000 3    60   ~ 0
+OUT-
+NoConn ~ 2250 5100
 $EndSCHEMATC
