File: Ardu2/design/POC-3_MAX395/KicadProjects/fullCircuit.kicad_pcb (KiCad board)
At the start: 4 copper layers, 240 x 188 mm, 126 parts, among them P1 CONN_01X02, P2 CONN_01X03, P3 CONN_01X03, P4 CONN_01X03, P5 CONN_01X03, P6 CONN_01X03, U1 Pyboard, U10 MAX395, U11 MAX395, U12 MAX395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

Commit message: progress on kicad design
Parts:
- removed U1: Pyboard, Socket_Strips:Socket_Strip_Straight_1x16
- added REF** (x2): Pyboard, 330L:Pyboard16x2, F.Cu at (45.7, 96.5)
Routing:
- net GND: track 973.0 -> 0.00 mm
- net /V+: track 560.1 -> 0.00 mm
- net /V-: track 557.4 -> 0.00 mm
- net Net-(U1-Pad4): track 374.1 -> 0.00 mm
- net Net-(U1-Pad6): track 357.9 -> 0.00 mm
- net /MIn+: track 214.2 -> 0.00 mm
- net /MIn-: track 211.5 -> 0.00 mm, vias 1 -> 0
- net /BOut-: track 190.3 -> 0.00 mm
- net /BATin: track 169.2 -> 0.00 mm, vias 1 -> 0
- net /DOut+: track 135.9 -> 0.00 mm
- net /BOut+: track 131.6 -> 0.00 mm
- net /COut-: track 121.3 -> 0.00 mm
- net /DOut-: track 114.0 -> 0.00 mm
- net /AOut-: track 110.3 -> 0.00 mm
- net /AOut+: track 105.2 -> 0.00 mm
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
Commit message: working 2 layer kicad pcb
Parts:
- removed P2, P3, P4, P5, P6: CONN_01X03, Connect:PINHEAD1-3
- removed REF** (x2): Pyboard, 330L:Pyboard16x2
- added HS1: HEATSINK, 330L:Heatsink_TO_220_38_20, F.Cu at (113.7, 123.2)
- added Hole1: MountingHole_3mm, Mounting_Holes:MountingHole_3mm, F.Cu at (73.7, 26.7)
- added Hole2: MountingHole_3mm, Mounting_Holes:MountingHole_3mm, F.Cu at (73.7, 141.0)
- added Hole3: MountingHole_3mm, Mounting_Holes:MountingHole_3mm, F.Cu at (224.8, 141.0)
- added P7: CONN_01X15, w_conn_pc:DB_15F-VGA, F.Cu at (222.2, 40.6)
- added U1: Pyboard, 330L:Pyboard16x2, F.Cu at (86.4, 95.2)
- U2, U3: footprint NationalSemiconductor:TO263-5 -> NationalSemiconductor:T05D
- moved L3 144.6 mm to (215.9, 58.4)
- moved L2 121.9 mm to (139.7, 127.0), turned to 90 degrees
- moved C2 100.0 mm to (118.1, 134.6)
- moved D2 93.9 mm to (128.3, 130.8), turned to 90 degrees
- moved R3 89.3 mm to (92.7, 101.6), turned to 180 degrees
- moved R2 84.6 mm to (92.7, 99.1)
- moved P1 73.0 mm to (73.7, 105.4), turned to 90 degrees
- moved C4 72.2 mm to (118.1, 113.0)
- moved L1 72.2 mm to (77.5, 121.9), turned to 270 degrees
- moved D1 70.3 mm to (94.0, 115.6), turned to 270 degrees
- moved U3 66.8 mm to (106.7, 123.2), turned to 270 degrees
- moved U4 60.9 mm to (100.3, 52.1)
- moved R1 58.3 mm to (99.1, 43.2)
- moved C3 53.9 mm to (85.1, 135.9), turned to 90 degrees
- moved C1 53.0 mm to (87.6, 113.0), turned to 90 degrees
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Connections:
- L3 pad 2: /MIn- -> Net-(L3-Pad2)
- U10 pad 24: Net-(U1-Pad4) -> Net-(U10-Pad24)
- U11 pad 24: Net-(U1-Pad4) -> Net-(U1-Pad5)
- U12 pad 24: Net-(U1-Pad4) -> Net-(U1-Pad5)
- U13 pad 24: Net-(U1-Pad4) -> Net-(U10-Pad24)
- U14 pad 24: Net-(U1-Pad4) -> Net-(U1-Pad5)
- U15 pad 24: Net-(U1-Pad4) -> Net-(U1-Pad5)
- U16 pad 24: Net-(U1-Pad4) -> Net-(U10-Pad24)
- U17 pad 24: Net-(U1-Pad4) -> Net-(U1-Pad5)
- U18 pad 24: Net-(U1-Pad4) -> Net-(U1-Pad5)
- U5 pad 24: Net-(U1-Pad4) -> Net-(U1-Pad5)
- U6 pad 24: Net-(U1-Pad4) -> Net-(U1-Pad5)
- U7 pad 22: Net-(U7-Pad22) -> (no net)
- U7 pad 24: Net-(U1-Pad4) -> Net-(U10-Pad24)
- U8 pad 24: Net-(U1-Pad4) -> Net-(U1-Pad5)
- U9 pad 24: Net-(U1-Pad4) -> Net-(U1-Pad5)
Routing:
- net GND: track 0.00 -> 559.0 mm
- net /V+: track 0.00 -> 415.9 mm
- net /V-: track 0.00 -> 410.6 mm
- net /MIn-: track 0.00 -> 283.8 mm, vias 0 -> 1
- net Net-(U1-Pad6): track 0.00 -> 268.8 mm
- net /MIn+: track 0.00 -> 200.0 mm
- net Net-(U1-Pad5): track 0.00 -> 153.6 mm
- net /OUT+: track 0.00 -> 152.0 mm
- net /BOut-: track 0.00 -> 149.9 mm
- net /DOut+: track 0.00 -> 130.8 mm
- net /DOut-: track 0.00 -> 107.3 mm
- net /COut-: track 0.00 -> 103.2 mm
- net /BOut+: track 0.00 -> 101.4 mm
- net /D-: track 0.00 -> 89.0 mm
- net /D+: track 0.00 -> 81.4 mm
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- added copper zone on B.Cu, net GND
- added copper zone on F.Cu, net GND
Other:
- board size 240 x 188 mm -> 163.8 x 125.7 mm
- copper layers 4 -> 2
- net class BATinput added: clearance 0.2, trace_width 0.3, via_dia 0.6, via_drill 0.4
- net class GND added: clearance 0.2, trace_width 0.3, via_dia 0.6, via_drill 0.4
- net class V+ added: clearance 0.2, trace_width 0.3, via_dia 0.6, via_drill 0.4
- net class V- added: clearance 0.2, trace_width 0.3, via_dia 0.6, via_drill 0.4

Commit message: ùore pcb kicad work, mostly failures
Parts:
- U4: value PHOTORESISTOR -> Vactrol; footprint Divers:OPTORESISTOR_NSL-32 -> 330L:Vactrol
- moved U4 8.47 mm to (92.1, 50.2)
- moved R1 0.63 mm to (99.1, 42.5)
Connections:
- net Net-(U1-Pad6) renamed /CLK
- U1 pad 1: Net-(U1-Pad1) -> /ShuntControl
- U1 pad 5: Net-(U1-Pad5) -> /CS
- U10 pad 24: Net-(U10-Pad24) -> /CS
- U11 pad 24: Net-(U1-Pad5) -> /CS
- U12 pad 24: Net-(U1-Pad5) -> /CS
- U13 pad 24: Net-(U10-Pad24) -> /CS
- U14 pad 24: Net-(U1-Pad5) -> /CS
- U15 pad 24: Net-(U1-Pad5) -> /CS
- U16 pad 24: Net-(U10-Pad24) -> /CS
- U17 pad 24: Net-(U1-Pad5) -> /CS
- U18 pad 24: Net-(U1-Pad5) -> /CS
- U4 pad 1: Net-(U1-Pad1) -> Net-(R1-Pad1)
- U4 pad 2: Net-(R1-Pad1) -> /ShuntControl
- U5 pad 24: Net-(U1-Pad5) -> /CS
- U6 pad 24: Net-(U1-Pad5) -> /CS
- U7 pad 24: Net-(U10-Pad24) -> /CS
- U8 pad 24: Net-(U1-Pad5) -> /CS
- U9 pad 24: Net-(U1-Pad5) -> /CS
Routing:
- net GND: track 559.0 -> 188.1 mm, vias 0 -> 1
- net /V-: track 410.6 -> 62.5 mm
- net /V+: track 415.9 -> 95.8 mm
- net /MIn-: track 283.8 -> 0.00 mm, vias 1 -> 0
- net /CLK: track 268.8 -> 0.00 mm
- net /MIn+: track 200.0 -> 0.00 mm
- net Net-(U1-Pad5): track 153.6 -> 0.00 mm
- net /OUT+: track 152.0 -> 0.00 mm
- net /BOut-: track 149.9 -> 0.00 mm
- net /DOut+: track 130.8 -> 0.00 mm
- net /DOut-: track 107.3 -> 0.00 mm
- net /COut-: track 103.2 -> 0.00 mm
- net /BOut+: track 101.4 -> 0.00 mm
- net /D-: track 89.0 -> 0.00 mm
- net /D+: track 81.4 -> 0.00 mm
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- removed copper zone on B.Cu, net GND
- removed copper zone on F.Cu, net GND
Other:
- net class Audio: clearance 0.2 -> 0.38; trace_width 0.12 -> 0.38
- net class BATinput: trace_width 0.3 -> 1.8
- net class GND: trace_width 0.3 -> 1.8
- net class Power: trace_width 0.3 -> 1.8
- net class SPI: clearance 0.2 -> 0.38; trace_width 0.12 -> 0.38
- net class V+: trace_width 0.3 -> 1.8
- net class V-: trace_width 0.3 -> 1.8

Commit message: more pcb experiments
Parts:
- moved P7 62.3 mm to (161.3, 27.9), turned to 180 degrees
- moved U4 48.0 mm to (135.9, 30.5)
- moved L3 39.9 mm to (184.2, 34.3), turned to 180 degrees
- moved R1 24.0 mm to (118.1, 27.9), turned to 180 degrees
- moved C22 12.8 mm to (174.0, 128.3)
- moved C28 12.8 mm to (186.7, 128.3)
- moved C15 12.8 mm to (161.3, 128.3)
- moved C3 12.8 mm to (86.4, 148.6)
- moved C36 12.8 mm to (199.4, 128.3)
- moved D1 12.8 mm to (95.2, 128.3)
- moved R4 12.8 mm to (133.3, 152.4)
- moved R5 12.8 mm to (133.3, 149.9)
- moved C1 12.8 mm to (88.9, 125.7)
- moved C16 12.8 mm to (128.3, 86.4)
- moved C18 12.8 mm to (130.8, 76.2)
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Connections:
- P7 pad 11: /A- -> /B-
- P7 pad 12: /A+ -> /B+
- P7 pad 13: /B+ -> /A-
- P7 pad 14: /B- -> /A+
Routing:
- net GND: track 188.1 -> 0.00 mm, vias 1 -> 0
- net /V+: track 95.8 -> 0.00 mm
- net /BATin: track 72.1 -> 0.00 mm, vias 1 -> 0
- net /V-: track 62.5 -> 0.00 mm
- net Net-(D1-Pad1): track 45.2 -> 0.00 mm
- net Net-(R4-Pad2): track 39.0 -> 0.00 mm
- net Net-(D2-Pad1): track 37.1 -> 0.00 mm
- net Net-(R2-Pad2): track 30.7 -> 0.00 mm
Other:
- board size 163.8 x 125.7 mm -> 162.6 x 133.3 mm
- net class Audio: clearance 0.38 -> 0.381; trace_width 0.38 -> 0.381
- net class BATinput: clearance 0.2 -> 0.381; trace_width 1.8 -> 0.762
- net class Default: clearance 0.2 -> 0.508; trace_width 0.25 -> 0.508
- net class GND: clearance 0.2 -> 0.381; trace_width 1.8 -> 0.762
- net class Power: clearance 0.2 -> 0.381; trace_width 1.8 -> 0.762
- net class SPI: clearance 0.38 -> 0.635; trace_width 0.38 -> 0.381
- net class V+: clearance 0.2 -> 0.381; trace_width 1.8 -> 0.762
- net class V-: clearance 0.2 -> 0.381; trace_width 1.8 -> 0.762
- rule trace_clearance: 0.2 -> 0.508

Commit message: another pcb version...
Parts:
- added Hole4: MountingHole_3mm, Mounting_Holes:MountingHole_3mm, F.Cu at (243.8, 22.9)
- moved C46 24.1 mm to (236.2, 86.4), turned to 180 degrees
- moved C41 21.6 mm to (218.4, 40.6)
- moved R47 21.6 mm to (238.8, 91.4)
- moved R48 21.6 mm to (238.8, 94.0)
- moved R49 21.6 mm to (238.8, 96.5)
- moved R50 21.6 mm to (238.8, 99.1)
- moved R51 21.6 mm to (238.8, 101.6)
- moved C42 20.3 mm to (219.7, 59.7), turned to 180 degrees
- moved C43 20.3 mm to (219.7, 76.2), turned to 180 degrees
- moved C44 20.3 mm to (232.4, 64.8), turned to 0 degrees
- moved C45 20.3 mm to (232.4, 81.3), turned to 0 degrees
- moved U17 20.3 mm to (226.1, 53.3)
- moved U18 20.3 mm to (226.1, 87.6)
- moved C39 19.1 mm to (208.3, 86.4), turned to 180 degrees
- moved R43 19.1 mm to (213.4, 44.5)
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Connections:
- L3 pad 2: Net-(L3-Pad2) -> /MIn-
- P7 pad 10: Net-(L3-Pad2) -> /MIn-
- P7 pad 6: Net-(L3-Pad2) -> /MIn-
- P7 pad 7: Net-(L3-Pad2) -> /MIn-
- P7 pad 8: Net-(L3-Pad2) -> /MIn-
- P7 pad 9: Net-(L3-Pad2) -> /MIn-
- U1 pad 1: /ShuntControl -> (no net)
- U1 pad 17: (no net) -> /ShuntControl
Routing:
- net /V-: track 0.00 -> 484.7 mm, vias 0 -> 4
- net /CLK: track 0.00 -> 349.3 mm, vias 0 -> 10
- net /CS: track 0.00 -> 345.4 mm, vias 0 -> 7
- net /MIn-: track 0.00 -> 293.2 mm, vias 0 -> 1
- net /MIn+: track 0.00 -> 220.0 mm, vias 0 -> 4
- net /BOut-: track 0.00 -> 176.8 mm
- net /DOut-: track 0.00 -> 156.4 mm, vias 0 -> 1
- net /DOut+: track 0.00 -> 151.7 mm, vias 0 -> 1
- net Net-(R14-Pad1): track 0.00 -> 146.4 mm, vias 0 -> 3
- net /COut-: track 0.00 -> 140.5 mm, vias 0 -> 1
- net /BOut+: track 0.00 -> 127.0 mm
- net Net-(U5-Pad22): track 0.00 -> 126.5 mm, vias 0 -> 1
- net Net-(R16-Pad2): track 0.00 -> 121.9 mm, vias 0 -> 1
- net Net-(C16-Pad1): track 0.00 -> 96.7 mm, vias 0 -> 1
- net /A+: track 0.00 -> 87.1 mm
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- added copper zone on B.Cu, net /V+
- added copper zone on F.Cu, net GND
Other:
- board size 162.6 x 133.3 mm -> 186.7 x 143.5 mm

Commit message: looking better and better
Parts:
- moved R1 1.63 mm to (118.1, 22.6)
Routing:
- net /BOut+: track 127.0 -> 129.2 mm
- net /CS: track 345.4 -> 347.4 mm
- net Net-(R1-Pad1): track 5.63 -> 4.39 mm
- net /V-: track 484.7 -> 485.8 mm
- net GND: track 35.6 -> 34.5 mm
- net Net-(C12-Pad2): track 50.5 -> 51.2 mm
- net /MIn+: track 220.0 -> 220.6 mm

Commit message: seems pretty good, again...
Parts:
- moved L3 6.87 mm to (179.7, 31.8), turned to 90 degrees
- moved C36 6.35 mm to (217.2, 128.3)
- moved U1 5.24 mm to (81.3, 97.8)
- moved C3 5.08 mm to (86.4, 143.5), turned to 0 degrees
- moved C40 5.08 mm to (229.9, 133.3), turned to 0 degrees
- moved U16 5.08 mm to (223.5, 121.9)
- moved Hole3 4.02 mm to (246.4, 156.2)
- moved C28 3.81 mm to (196.8, 128.3)
- moved C35 3.81 mm to (209.6, 133.3)
- moved U13 3.81 mm to (203.2, 121.9)
- moved R1 2.55 mm to (115.6, 22.9)
- moved R38 2.54 mm to (213.4, 91.4)
- moved R39 2.54 mm to (213.4, 94.0)
- moved R40 2.54 mm to (213.4, 96.5)
- moved R41 2.54 mm to (213.4, 99.1)
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Connections:
- C31 pad 2: /BOut- -> /COut+
- U1 pad 30: (no net) -> GND
- U1 pad 32: (no net) -> /V+
- U10 pad 12: /BOut- -> /COut+
- U10 pad 16: /BOut- -> /COut+
- U10 pad 17: /BOut- -> /COut+
- U12 pad 10: /BOut- -> /COut+
- U12 pad 11: /BOut- -> /COut+
- U12 pad 13: /BOut- -> /COut+
- U12 pad 15: /BOut- -> /COut+
- U12 pad 18: /BOut- -> /COut+
- U12 pad 19: /BOut- -> /COut+
- U13 pad 9: /BOut- -> /COut+
- U16 pad 8: /BOut- -> /COut+
- U7 pad 20: /BOut- -> /COut+
- U7 pad 5: /BOut- -> /COut+
Routing:
- net /COut+: track 0.00 -> 217.3 mm, vias 0 -> 1
- net Net-(R14-Pad1): track 146.4 -> 62.0 mm, vias 3 -> 0
- net Net-(C16-Pad1): track 96.7 -> 36.1 mm, vias 1 -> 0
- net Net-(R16-Pad2): track 121.9 -> 61.5 mm, vias 1 -> 0
- net /V-: track 485.8 -> 540.5 mm
- net Net-(R17-Pad2): track 64.8 -> 118.0 mm, vias 0 -> 1
- net /BOut-: track 176.8 -> 128.0 mm, vias 0 -> 1
- net Net-(U12-Pad3): track 86.6 -> 40.9 mm, vias 3 -> 2
- net GND: track 34.5 -> 1.00 mm
- net /CS: track 347.4 -> 323.0 mm, vias 7 -> 8
- net Net-(C13-Pad2): track 30.6 -> 54.1 mm, vias 2 -> 0
- net /MIn+: track 220.6 -> 243.0 mm, vias 4 -> 3
- net /CLK: track 349.3 -> 328.1 mm, vias 10 -> 7
- net /COut-: track 140.5 -> 161.2 mm
- net /DOut-: track 156.4 -> 176.1 mm
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Other:
- board size 186.7 x 143.5 mm -> 189.2 x 143.5 mm
- net class BATinput: clearance 0.381 -> 0.254
- net class GND: clearance 0.381 -> 0.254
- net class Power: clearance 0.381 -> 0.254
- net class V+: clearance 0.381 -> 0.254
- net class V-: clearance 0.381 -> 0.254
