File: Ardu2/design/POC-3_MAX395/HMI/KicadProjects/HMI.kicad_pcb (KiCad board)
At the start: 2 copper layers, 0 parts

Commit message: HMI LED PCB 00
Parts:
- added C1: 100nF, Capacitors_ThroughHole:C_Disc_D3_P2.5, F.Cu at (128.9, 30.5)
- added C2: 100nF, Capacitors_ThroughHole:C_Disc_D3_P2.5, F.Cu at (127.7, 57.0)
- added C3: 100nF, Capacitors_ThroughHole:C_Disc_D3_P2.5, F.Cu at (128.3, 82.6)
- added C4: 100nF, Capacitors_ThroughHole:C_Disc_D3_P2.5, F.Cu at (125.7, 108.1)
- added C5: 100nF, Capacitors_ThroughHole:C_Disc_D3_P2.5, F.Cu at (124.4, 133.4)
- added H0: MountingHole_3mm, Mounting_Holes:MountingHole_3mm, F.Cu at (113.2, 30.5)
- added H1: MountingHole_3mm, Mounting_Holes:MountingHole_3mm, F.Cu at (164.0, 30.6)
- added H2: MountingHole_3mm, Mounting_Holes:MountingHole_3mm, F.Cu at (164.1, 150.1)
- added H3: MountingHole_3mm, Mounting_Holes:MountingHole_3mm, F.Cu at (114.1, 150.6)
- added P1: CONN_01X03, Pin_Headers:Pin_Header_Straight_1x03, F.Cu at (128.9, 36.7)
- added P10: CONN_01X02, Pin_Headers:Pin_Header_Straight_1x02, F.Cu at (127.4, 62.8)
- added P11: CONN_01X02, Pin_Headers:Pin_Header_Straight_1x02, F.Cu at (124.2, 139.2)
- added P12: CONN_01X02, Pin_Headers:Pin_Header_Straight_1x02, F.Cu at (125.1, 36.8)
- added P13: CONN_01X02, Pin_Headers:Pin_Header_Straight_1x02, F.Cu at (127.6, 88.5)
- added P14: CONN_01X02, Pin_Headers:Pin_Header_Straight_1x02, F.Cu at (125.2, 113.9)
- added P15: CONN_01X01, Pin_Headers:Pin_Header_Straight_1x01, F.Cu at (125.2, 120.7)
- added P16: CONN_01X01, Pin_Headers:Pin_Header_Straight_1x01, F.Cu at (124.2, 146.1)
- added P17: CONN_01X01, Pin_Headers:Pin_Header_Straight_1x01, F.Cu at (127.6, 69.6)
- added P18: CONN_01X01, Pin_Headers:Pin_Header_Straight_1x01, F.Cu at (127.7, 95.3)
- added P19: CONN_01X01, Pin_Headers:Pin_Header_Straight_1x01, F.Cu at (124.4, 129.0)
- added P2: CONN_01X02, Pin_Headers:Pin_Header_Straight_1x02, F.Cu at (128.7, 48.4)
- added P3: CONN_02X20, Pin_Headers:Pin_Header_Straight_2x20, F.Cu at (164.6, 39.9)
- added P4: CONN_02X20, Pin_Headers:Pin_Header_Straight_2x20, F.Cu at (164.6, 93.5)
- added P5: CONN_01X02, Pin_Headers:Pin_Header_Straight_1x02, F.Cu at (112.7, 39.3)
- added P6: CONN_01X03, Pin_Headers:Pin_Header_Straight_1x03, F.Cu at (110.1, 69.7)
- added P7: CONN_01X03, Pin_Headers:Pin_Header_Straight_1x03, F.Cu at (110.1, 95.2)
- added P8: CONN_01X03, Pin_Headers:Pin_Header_Straight_1x03, F.Cu at (110.1, 120.6)
- added P9: CONN_01X03, Pin_Headers:Pin_Header_Straight_1x03, F.Cu at (110.1, 141.7)
- added R1: 1K, Resistors_ThroughHole:Resistor_Horizontal_RM10mm, F.Cu at (154.6, 39.9)
- added R10: 1K, Resistors_ThroughHole:Resistor_Horizontal_RM10mm, F.Cu at (154.6, 62.8)
- added R11: 1K, Resistors_ThroughHole:Resistor_Horizontal_RM10mm, F.Cu at (154.6, 65.3)
- added R12: 1K, Resistors_ThroughHole:Resistor_Horizontal_RM10mm, F.Cu at (154.6, 67.8)
- added R13: 1K, Resistors_ThroughHole:Resistor_Horizontal_RM10mm, F.Cu at (154.6, 70.4)
- added R14: 1K, Resistors_ThroughHole:Resistor_Horizontal_RM10mm, F.Cu at (154.6, 72.9)
- added R15: 1K, Resistors_ThroughHole:Resistor_Horizontal_RM10mm, F.Cu at (154.6, 75.4)
- added R16: 1K, Resistors_ThroughHole:Resistor_Horizontal_RM10mm, F.Cu at (154.6, 78.0)
- added R17: 1K, Resistors_ThroughHole:Resistor_Horizontal_RM10mm, F.Cu at (154.6, 80.5)
- added R18: 1K, Resistors_ThroughHole:Resistor_Horizontal_RM10mm, F.Cu at (154.6, 83.1)
- added R19: 1K, Resistors_ThroughHole:Resistor_Horizontal_RM10mm, F.Cu at (154.6, 85.6)
- added R2: 1K, Resistors_ThroughHole:Resistor_Horizontal_RM10mm, F.Cu at (154.6, 42.4)
- added R20: 1K, Resistors_ThroughHole:Resistor_Horizontal_RM10mm, F.Cu at (154.6, 88.1)
- added R21: 1K, Resistors_ThroughHole:Resistor_Horizontal_RM10mm, F.Cu at (154.6, 93.5)
- added R22: 1K, Resistors_ThroughHole:Resistor_Horizontal_RM10mm, F.Cu at (154.6, 96.0)
- added R23: 1K, Resistors_ThroughHole:Resistor_Horizontal_RM10mm, F.Cu at (154.6, 98.6)
- added R24: 1K, Resistors_ThroughHole:Resistor_Horizontal_RM10mm, F.Cu at (154.6, 101.1)
- added R25: 1K, Resistors_ThroughHole:Resistor_Horizontal_RM10mm, F.Cu at (154.6, 103.6)
- added R26: 1K, Resistors_ThroughHole:Resistor_Horizontal_RM10mm, F.Cu at (154.6, 106.2)
- added R27: 1K, Resistors_ThroughHole:Resistor_Horizontal_RM10mm, F.Cu at (154.6, 108.7)
- added R28: 1K, Resistors_ThroughHole:Resistor_Horizontal_RM10mm, F.Cu at (154.6, 111.3)
- added R29: 1K, Resistors_ThroughHole:Resistor_Horizontal_RM10mm, F.Cu at (154.6, 113.8)
- added R3: 1K, Resistors_ThroughHole:Resistor_Horizontal_RM10mm, F.Cu at (154.6, 45.0)
- added R30: 1K, Resistors_ThroughHole:Resistor_Horizontal_RM10mm, F.Cu at (154.6, 116.3)
- added R31: 1K, Resistors_ThroughHole:Resistor_Horizontal_RM10mm, F.Cu at (154.6, 118.9)
- added R32: 1K, Resistors_ThroughHole:Resistor_Horizontal_RM10mm, F.Cu at (154.6, 121.4)
- added R33: 1K, Resistors_ThroughHole:Resistor_Horizontal_RM10mm, F.Cu at (154.6, 124.0)
- added R34: 1K, Resistors_ThroughHole:Resistor_Horizontal_RM10mm, F.Cu at (154.6, 126.5)
- added R35: 1K, Resistors_ThroughHole:Resistor_Horizontal_RM10mm, F.Cu at (154.6, 129.1)
- added R36: 1K, Resistors_ThroughHole:Resistor_Horizontal_RM10mm, F.Cu at (154.6, 131.6)
- added R37: 1K, Resistors_ThroughHole:Resistor_Horizontal_RM10mm, F.Cu at (154.6, 134.1)
- added R4: 1K, Resistors_ThroughHole:Resistor_Horizontal_RM10mm, F.Cu at (154.6, 47.5)
- added R5: 1K, Resistors_ThroughHole:Resistor_Horizontal_RM10mm, F.Cu at (154.6, 50.0)
- added R6: 1K, Resistors_ThroughHole:Resistor_Horizontal_RM10mm, F.Cu at (154.6, 52.6)
- added R7: 1K, Resistors_ThroughHole:Resistor_Horizontal_RM10mm, F.Cu at (154.6, 55.1)
- added R8: 1K, Resistors_ThroughHole:Resistor_Horizontal_RM10mm, F.Cu at (154.6, 57.7)
- added R9: 1K, Resistors_ThroughHole:Resistor_Horizontal_RM10mm, F.Cu at (154.6, 60.2)
- added U1: 74HC595, Housings_DIP:DIP-16_W7.62mm, F.Cu at (137.2, 125.7)
- added U2: 74HC595, Housings_DIP:DIP-16_W7.62mm, F.Cu at (139.0, 74.7)
- added U3: 74HC595, Housings_DIP:DIP-16_W7.62mm, F.Cu at (135.5, 151.2)
- added U4: 74HC595, Housings_DIP:DIP-16_W7.62mm, F.Cu at (140.7, 49.3)
- added U5: 74HC595, Housings_DIP:DIP-16_W7.62mm, F.Cu at (139.5, 100.4)
Routing:
- net /CLK: track 0.00 -> 223.2 mm
- net /LATCH: track 0.00 -> 205.5 mm
- net +5V: track 0.00 -> 192.9 mm
- net GND: track 0.00 -> 103.5 mm
- net Net-(P17-Pad1): track 0.00 -> 72.3 mm
- net Net-(P18-Pad1): track 0.00 -> 68.3 mm
- net Net-(P15-Pad1): track 0.00 -> 66.2 mm
- net Net-(P16-Pad1): track 0.00 -> 62.0 mm
- net /UU2: track 0.00 -> 43.8 mm
- net /UU0: track 0.00 -> 34.0 mm
- net /UU1: track 0.00 -> 34.0 mm
- net /TR1: track 0.00 -> 24.9 mm
- net /DT2: track 0.00 -> 22.2 mm
- net /BV1: track 0.00 -> 20.9 mm
- net /CT0: track 0.00 -> 20.6 mm
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- added copper zone on B.Cu, net GND
Other:
- board outline added: 65.3 x 131.6 mm
- net class Default: clearance 0.2 -> 0.5; trace_width 0.25 -> 1
- net class Power added: clearance 0.5, trace_width 1.3, via_dia 0.6, via_drill 0.4
- net class SPI added: clearance 0.5, trace_width 1, via_dia 0.6, via_drill 0.4
- rule trace_clearance: 0.2 -> 0.5

Commit message: HMI PCB v2a
Parts:
- added R38: 1K, Resistors_ThroughHole:Resistor_Horizontal_RM10mm, F.Cu at (154.6, 137.4)
- added R39: 1K, Resistors_ThroughHole:Resistor_Horizontal_RM10mm, F.Cu at (154.6, 140.6)
- added R40: 1K, Resistors_ThroughHole:Resistor_Horizontal_RM10mm, F.Cu at (154.6, 143.8)
- moved H1 5.32 mm to (169.3, 30.7)
- moved H2 5.31 mm to (169.1, 152.0)
- moved H3 3.12 mm to (111.4, 152.0)
- moved H0 1.78 mm to (111.4, 30.7)
Connections:
- P4 pad 35: /UU0 -> Net-(P4-Pad35)
- P4 pad 37: /UU1 -> Net-(P4-Pad37)
- P4 pad 39: /UU2 -> Net-(P4-Pad39)
Routing:
- net GND: track 103.5 -> 120.0 mm
- net /UU2: track 43.8 -> 27.9 mm
- net /UU1: track 34.0 -> 18.4 mm
- net /UU0: track 34.0 -> 18.7 mm
- net Net-(P4-Pad39): track 0.00 -> 5.33 mm
- net Net-(P4-Pad37): track 0.00 -> 5.12 mm
- net Net-(P4-Pad35): track 0.00 -> 4.98 mm
Other:
- board size 65.3 x 131.6 mm -> 68.7 x 131.6 mm
- board text added: "AT0"
- board text added: "AT1"
- board text added: "AT2"
- board text added: "AV0"
- board text added: "AV1"
- board text added: "AV2"
- board text added: "BT0"
- board text added: "BT1"
- board text added: "BT2"
- board text added: "BV0"
- board text added: "BV1"
- board text added: "BV2"
- board text added: "CT0"
- board text added: "CT1"
- board text added: "CT2"
- board text added: "CV0"
- board text added: "CV1"
- board text added: "CV2"
- board text added: "DT0"
- board text added: "DT1"
- board text added: "DT2"
- board text added: "DV0"
- board text added: "DV1"
- board text added: "DV2"
- board text added: "HMI Bottom Layer"
- board text added: "MT0"
- board text added: "MT1"
- board text added: "MT2"
- board text added: "MV0"
- board text added: "MV1"
- board text added: "MV2"
- board text added: "PBLL"
- board text added: "PBLR"
- board text added: "PBUL"
- board text added: "PBUR"
- board text added: "TR0"
- board text added: "TR1"
- board text added: "TR2"
- board text added: "UU0"
- board text added: "UU1"
- board text added: "UU2"
