File: Ardu2/design/POC-3_MAX395/HMI/KicadProjects/2PB with Headers/2PB with Headers.kicad_pcb (KiCad board)
At the start: 2 copper layers, 44.7 x 11.4 mm, 5 parts, among them SW1 SW_PUSH, SW2 SW_PUSH

Commit message: PB PCB work
Parts:
- GND P2 P1: footprint Pin_Headers:Pin_Header_Straight_1x03 -> misc:Pin_Header_Straight_1x03
