File: Ardu2/design/POC-3_MAX395/HMI/KicadProjects/Multi-PB-Debounce Circuit/Multi-PB-Debounce Circuit.kicad_pcb (KiCad board)
At the start: 2 copper layers, 76.2 x 26.7 mm, 23 parts

Commit message: PB PCB work
Parts:
- C1, C2, C3, C4, C5, C6: footprint Capacitors_ThroughHole:C_Radial_D5_L11_P2 -> misc:C_Radial_D5_L11_P2
- GND, SW: footprint Pin_Headers:Pin_Header_Straight_1x06 -> misc:Pin_Header_Straight_1x06
- GND Pins VCC: footprint Pin_Headers:Pin_Header_Straight_1x08 -> misc:Pin_Header_Straight_1x08
