File: Ardu2/design/POC-3_MAX395/HMI/KicadProjects/Main HMI Circuit/HMI.kicad_pcb (KiCad board)
At the start: 2 copper layers, 68.7 x 131.6 mm, 73 parts, among them P1 CONN_01X03, P10 CONN_01X02, P11 CONN_01X02, P12 CONN_01X02, P13 CONN_01X02, P14 CONN_01X02, P15 CONN_01X01, P16 CONN_01X01, P17 CONN_01X01, P18 CONN_01X01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

Commit message: working on the HMI LEDs
Parts:
- renumbered U3 to U0, U5 to U2, U2 to U3
Changed lines of the file:
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@@
-(kicad_pcb (version 4) (host pcbnew 0.201511171411+6319~30~ubuntu15.04.1-product)
+(kicad_pcb (version 4) (host pcbnew 4.1.0-alpha+201605292346+6852~44~ubuntu15.10.1-product)
   (general
     (links 194)
     (no_connects 0)
-    (area 104.590474 25.2577 178.081046 158.32066)
+    (area 104.590475 25.4252 178.081046 158.43816)
     (thickness 1.6)
     (drawings 48)
@@
       (hpglpenspeed 20)
       (hpglpendiameter 15)
-      (hpglpenoverlay 2)
       (psnegative false)
       (psa4output false)
@@
     (descr "16-lead dip package, row spacing 7.62 mm (300 mils)")
     (tags "dil dip 2.54 300")
-    (fp_text reference U2 (at 3.9624 8.7376 180) (layer F.SilkS)
+    (fp_text reference U3 (at 3.9624 8.7376 180) (layer F.SilkS)
       (effects (font (size 1 1) (thickness 0.15)))
     )
@@
     (descr "16-lead dip package, row spacing 7.62 mm (300 mils)")
     (tags "dil dip 2.54 300")
-    (fp_text reference U3 (at 3.9624 8.7884 180) (layer F.SilkS)
+    (fp_text reference U0 (at 3.9624 8.7884 180) (layer F.SilkS)
       (effects (font (size 1 1) (thickness 0.15)))
     )
@@
     (descr "16-lead dip package, row spacing 7.62 mm (300 mils)")
     (tags "dil dip 2.54 300")
-    (fp_text reference U5 (at 3.9624 7.1374 180) (layer F.SilkS)
+    (fp_text reference U2 (at 3.9624 7.1374 180) (layer F.SilkS)
       (effects (font (size 1 1) (thickness 0.15)))
     )
@@
     (descr "Through hole pin header")
     (tags "pin header")
-    (fp_text reference P5 (at -2.794 2.54 360) (layer F.SilkS)
-      (effects (font (size 1 1) (thickness 0.15)))
-    )
+    (fp_text reference P5 (at -2.794 2.54) (layer F.SilkS)
+      (effects (font (size 1 1) (thickness 0.15)))
+    )
