File: Ardu2/design/POC-3_MAX395/HMI/KicadProjects/Main HMI Circuit/HMI.sch (KiCad schematic (older format))
At the start: 69 parts, among them P1 CONN_01X03, P10 CONN_01X02, P11 CONN_01X02, P12 CONN_01X02, P13 CONN_01X02, P14 CONN_01X02, P15 CONN_01X01, P16 CONN_01X01, P17 CONN_01X01, P18 CONN_01X01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

Commit message: working on the HMI LEDs
Parts:
- renumbered U3 to U0, U5 to U2, U2 to U3
Changed lines of the file:
@@
 GND
 $Comp
-L 74HC595 U5
+L 74HC595 U2
 U 1 1 564C135D
 P 4870 5120
-F 0 "U5" H 5020 5720 70  0000 C CNN
+F 0 "U2" H 5020 5720 70  0000 C CNN
 F 1 "74HC595" H 4870 4520 70  0000 C CNN
 F 2 "Housings_DIP:DIP-16_W7.62mm" H 4870 5120 60  0001 C CNN
@@
 Vcc
 $Comp
-L 74HC595 U2
+L 74HC595 U3
 U 1 1 564C4B0F
 P 4830 3620
-F 0 "U2" H 4980 4220 70  0000 C CNN
+F 0 "U3" H 4980 4220 70  0000 C CNN
 F 1 "74HC595" H 4830 3020 70  0000 C CNN
 F 2 "Housings_DIP:DIP-16_W7.62mm" H 4830 3620 60  0001 C CNN
@@
 Vcc
 $Comp
-L 74HC595 U3
+L 74HC595 U0
 U 1 1 564C517A
 P 4830 8080
-F 0 "U3" H 4980 8680 70  0000 C CNN
+F 0 "U0" H 4980 8680 70  0000 C CNN
 F 1 "74HC595" H 4830 7480 70  0000 C CNN
 F 2 "Housings_DIP:DIP-16_W7.62mm" H 4830 8080 60  0001 C CNN
