File: Ardu2/design/POC-3_MAX395/KicadProjects/HMI_PCB/HMI-PCB.kicad_pcb (KiCad board)
At the start: 2 copper layers, 170.2 x 72.9 mm, 52 parts, among them P1 SplitPot_0_M, P10 TREM_VIB, P11 SplitPot_5_TR, P12 Analog Power IN, P13 Digital Power IN/OUT, P2 SEQ_SAVE, P3 SplitPot_1_A, P4 SplitPot_2_B, P5 PB_OUT, P6 Analog_Signal_Out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

Commit message: final update to HMI PCB
Parts:
- C1, C2, C3, C4, C5, C6: footprint misc:C_Radial_D5_L11_P3.81_pads_2_mm_holes_7mm -> misc:C_Radial_D5_L11_P3.81
- C10, C11, C12, C7, C8, C9: footprint misc:C_Disc_D6_P5_2mm_Pad_0_7mm_hole -> Capacitors_ThroughHole:C_Disc_D6_P5
- C14: footprint Capacitors_ThroughHole:C_Radial_D5_L11_P2.5 -> Capacitors_ThroughHole:C_Disc_D3_P2.5
- C16: footprint Capacitors_ThroughHole:C_Radial_D5_L6_P2.5 -> Capacitors_ThroughHole:C_Disc_D3_P2.5
- L1: footprint Resistors_ThroughHole:Resistor_Horizontal_RM10mm -> misc:Choke_Radial_D13_P10_10mH
- moved C13 18.2 mm to (74.4, 108.0), turned to 90 degrees
- moved C16 11.2 mm to (77.0, 105.5), turned to 270 degrees
- moved C14 7.37 mm to (79.5, 105.5), turned to 270 degrees
- moved P6 7.37 mm to (86.4, 124.8)
- moved L1 3.69 mm to (77.5, 96.4), turned to 270 degrees
Routing:
- net /GND_A: track 259.9 -> 274.5 mm
- net /X3: track 85.1 -> 93.1 mm
- net /X4: track 110.4 -> 118.4 mm
- net /X1: track 19.5 -> 26.9 mm
- net /X2: track 56.5 -> 63.9 mm
- net /Y11: track 134.7 -> 141.7 mm
- net /Y12: track 169.1 -> 175.3 mm
- net /3v3_A: track 185.7 -> 183.6 mm
- net /3v3_A_IN: track 3.43 -> 4.88 mm
