File: Ardu2/design/POC-3_MAX395/KicadProjects/HMI_PCB/HMI-PCB.sch (KiCad schematic (older format))
At the start: 48 parts, among them P1 SplitPot_0_M, P10 TREM_VIB, P11 SplitPot_5_TR, P12 Analog Power IN, P13 Digital Power IN/OUT, P2 SEQ_SAVE, P3 SplitPot_1_A, P4 SplitPot_2_B, P5 PB_OUT, P6 Analog_Signal_Out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

Commit message: final update to HMI PCB
Parts:
- C14: footprint Capacitors_ThroughHole:C_Radial_D5_L11_P2.5 -> Capacitors_ThroughHole:C_Disc_D3_P2.5
- C16: footprint Capacitors_ThroughHole:C_Radial_D5_L6_P2.5 -> Capacitors_ThroughHole:C_Disc_D3_P2.5
- L1: footprint Resistors_ThroughHole:Resistor_Horizontal_RM10mm -> misc:Choke_Radial_D13_P10_10mH
Changed lines of the file:
@@
 F 0 "C14" V 5980 3510 50  0000 C CNN
 F 1 "10µF" V 5840 3220 50  0000 C CNN
-F 2 "Capacitors_ThroughHole:C_Radial_D5_L11_P2.5" H 5938 3260 50  0001 C CNN
+F 2 "Capacitors_ThroughHole:C_Disc_D3_P2.5" H 5938 3260 50  0001 C CNN
 F 3 "" H 5900 3410 50  0000 C CNN
 	1    5900 3410
@@
 F 0 "L1" V 5550 3640 50  0000 C CNN
 F 1 "10mH" V 5670 3620 50  0000 C CNN
-F 2 "Resistors_ThroughHole:Resistor_Horizontal_RM10mm" H 5590 3630 50  0001 C CNN
+F 2 "misc:Choke_Radial_D13_P10_10mH" H 5590 3630 50  0001 C CNN
 F 3 "" H 5590 3630 50  0000 C CNN
 	1    5590 3630
@@
 F 0 "C16" V 5850 3540 50  0000 C CNN
 F 1 "1µF" V 5950 3780 50  0000 C CNN
-F 2 "Capacitors_ThroughHole:C_Radial_D5_L6_P2.5" H 5938 3480 50  0001 C CNN
+F 2 "Capacitors_ThroughHole:C_Disc_D3_P2.5" H 5938 3480 50  0001 C CNN
 F 3 "" H 5900 3630 50  0000 C CNN
 	1    5900 3630
