File: Ardu3/Concept/Kicad/Unity Gain Digipot Vol-tone/Unity Gain Digipot Vol-tone.sch (KiCad schematic (older format))
At the start: 9 parts

Commit message: draft schematic for unity gain vol tone
Connections:
- wire segments 33 -> 31
Changed lines of the file:
@@
 F 3 "" H 2990 3790 50  0001 C CNN
 	2    2990 3790
-	1    0    0    1
+	1    0    0    -1
 $EndComp
-Wire Wire Line
-	3260 3690 3190 3690
-Wire Wire Line
-	3330 3890 3190 3890
 Wire Wire Line
 	2490 3380 2790 3380
@@
 Wire Wire Line
 	2790 3880 2790 3790
-Wire Wire Line
-	8380 5390 3330 5390
-Wire Wire Line
-	3330 5390 3330 3890
-Connection ~ 3330 3890
-Wire Wire Line
-	3190 3380 3260 3380
-Wire Wire Line
-	3260 3690 3260 3380
-Connection ~ 3260 3380
-Wire Wire Line
-	3260 3380 4140 3380
-Wire Wire Line
-	3190 3580 3330 3580
-Wire Wire Line
-	3330 3580 3330 3890
-Wire Wire Line
-	3330 3890 3330 3900
 Wire Notes Line
 	2740 4100 3450 4100
@@
 Inverter
 NoConn ~ 6620 3180
+Wire Wire Line
+	3190 3380 3270 3380
+Wire Wire Line
+	3190 3580 3190 3690
+Wire Wire Line
+	3190 3890 3270 3890
+Wire Wire Line
+	3270 3890 3270 3380
+Connection ~ 3270 3380
+Wire Wire Line
+	3270 3380 4140 3380
+Wire Wire Line
+	8380 5390 3330 5390
+Wire Wire Line
+	3330 5390 3330 3690
+Wire Wire Line
+	3330 3690 3190 3690
+Connection ~ 3190 3690
 $EndSCHEMATC

Commit message: more work on digipot vol tone
Parts:
- added C? (x2): 20pF, symbol Device:C
- added R? (x2): 1M, symbol Device:R
- added U? (x2): LM1875, Package_TO_SOT_THT:TO-220-5_Vertical_StaggeredType1_Py3.7mm, symbol Amplifier_Audio:LM1875
Connections:
- wire segments 31 -> 61
- no-connect marks 1 -> 0
